Commit message: lidar bug fix

File: gem_description/urdf/gem.urdf.xacro (robot description, xacro)
@@ -1202,5 +1202,5 @@
   </link>
   <joint name="velodyne_joint" type="fixed">
-    <origin xyz="0.02 0.115 -0.6575" rpy="1.5708 0 3.1416" />
+    <origin xyz="0.02 0.15 -0.6575" rpy="1.5708 0 3.1416" />
     <parent link="top_rack_link"/>
     <child link="velodyne_link"/>
@@ -1212,4 +1212,5 @@
       <visualize>false</visualize>
       <update_rate>10</update_rate>
+      <always_on>true</always_on>
       <lidar>
         <scan>
@@ -1238,5 +1239,5 @@
         </noise>
       </lidar>
-      <topic>scan</topic>
+      <topic>/scan</topic>
       <gz_frame_id>velodyne_link</gz_frame_id>
     </sensor>
